File: microstrip/microstrip.kicad_sch (KiCad schematic)
At the start: 0 parts

Commit message: Adicionando arquivos de design do KiCAD.
Other:
- company: (none) -> Eng. Ygor K.
- title: (none) -> Microstrip
Changed lines of the file:
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@@
 	(generator_version "9.0")
 	(paper "A4")
+	(title_block
+		(title "Microstrip")
+		(company "Eng. Ygor K.")
+	)
 	(sheet_instances
 		(path "/"

Commit message: Designed and exported to .step file.
Other:
- title: Microstrip -> Microstrip Coplanar Waveguide
